File: RP2350 Dev Board.kicad_sch (KiCad schematic)
At the start: 60 parts, among them J1 Conn_01x32_MountingPin, J2 Conn_01x03_Pin, J3 Conn_01x32_MountingPin, U4 Winbond W25Q128JVSIQ, U5 RPI Radio Module 2, U6 ESP-PSRAM32

Commit message: final cleanup
Connections:
- net 3V3: now also J1.28 (60); no longer J1.60 (Pin_60)
- net 3V3_EN: now also J1.29 (61); no longer J1.61 (Pin_61)
- net ADC_VREF: now also J1.27 (59); no longer J1.59 (Pin_59)
- net GND: now also J1.15 (47), J1.2 (34), J1.20 (52), J1.25 (57), J1.30 (62); no longer J1.34 (Pin_34), J1.47 (Pin_47), J1.52 (Pin_52), J1.57 (Pin_57), J1.62 (Pin_62)
- net GPIO16: now also J1.13 (45); no longer J1.45 (Pin_45)
- net GPIO17: now also J1.14 (46); no longer J1.46 (Pin_46)
- net GPIO18: now also J1.16 (48); no longer J1.48 (Pin_48)
- net GPIO19: now also J1.17 (49); no longer J1.49 (Pin_49)
- net GPIO20: now also J1.18 (50); no longer J1.50 (Pin_50)
- net GPIO21: now also J1.19 (51); no longer J1.51 (Pin_51)
- net GPIO22: now also J1.21 (53); no longer J1.53 (Pin_53)
- net GPIO26: now also J1.23 (55); no longer J1.55 (Pin_55)
- net GPIO27: now also J1.24 (56); no longer J1.56 (Pin_56)
- net GPIO28: now also J1.26 (58); no longer J1.58 (Pin_58)
- net GPIO37: now also J1.1 (33); no longer J1.33 (Pin_33)
- net GPIO38: now also J1.3 (35); no longer J1.35 (Pin_35)
- net GPIO39: now also J1.4 (36); no longer J1.36 (Pin_36)
- net GPIO40/ADC0: now also J1.5 (37); no longer J1.37 (Pin_37)
- net GPIO41/ADC1: now also J1.6 (38); no longer J1.38 (Pin_38)
- net GPIO42/ADC2: now also J1.7 (39); no longer J1.39 (Pin_39)
- net GPIO43/ADC3: now also J1.8 (40); no longer J1.40 (Pin_40)
- net GPIO44/ADC4: now also J1.9 (41); no longer J1.41 (Pin_41)
- net GPIO45/ADC5: now also J1.10 (42); no longer J1.42 (Pin_42)
- net GPIO46/ADC6: now also J1.11 (43); no longer J1.43 (Pin_43)
- net GPIO47/ADC7: now also J1.12 (44); no longer J1.44 (Pin_44)
- net RUN: now also J1.22 (54); no longer J1.54 (Pin_54)
- net VBUS: now also J1.32 (64); no longer J1.64 (Pin_64)
- net VSYS: now also J1.31 (63); no longer J1.63 (Pin_63)
Changed lines of the file:
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@@
 			)
 		)
-		(pin "33"
+		(pin "32"
 		)
-		(pin "34"
+		(pin "31"
 		)
-		(pin "35"
+		(pin "30"
 		)
-		(pin "36"
+		(pin "29"
 		)
-		(pin "37"
+		(pin "28"
 		)
-		(pin "38"
+		(pin "27"
 		)
-		(pin "39"
+		(pin "26"
 		)
-		(pin "40"
+		(pin "25"
 		)
-		(pin "41"
+		(pin "24"
 		)
-		(pin "42"
+		(pin "23"
 		)
-		(pin "43"
+		(pin "22"
 		)
-		(pin "44"
+		(pin "21"
 		)
-		(pin "45"
+		(pin "20"
 		)
-		(pin "46"
+		(pin "19"
 		)
-		(pin "47"
+		(pin "18"
 		)
-		(pin "48"
+		(pin "17"
 		)
-		(pin "49"
+		(pin "16"
 		)
-		(pin "50"
+		(pin "15"
 		)
-		(pin "51"
+		(pin "14"
 		)
-		(pin "52"
+		(pin "13"
 		)
-		(pin "53"
+		(pin "12"
 		)
-		(pin "54"
+		(pin "11"
 		)
-		(pin "55"
+		(pin "10"
 		)
-		(pin "56"
+		(pin "9"
 		)
-		(pin "57"
+		(pin "8"
 		)
-		(pin "58"
+		(pin "7"
 		)
-		(pin "59"
+		(pin "6"
 		)
-		(pin "60"
+		(pin "5"
 		)
-		(pin "61"
+		(pin "4"
 		)
-		(pin "62"
+		(pin "3"
 		)
-		(pin "63"
+		(pin "2"
 		)
-		(pin "64"
+		(pin "1"
 		)
 		(pin "MP"

Commit message: Before RM2 reset
Parts:
- added TP1, TP2: TestPoint, TestPoint:TestPoint_Pad_1.0x1.0mm, symbol Connector:TestPoint
Connections:
- net 1V1: now also TP1.1
- net 3V3: now also C16.1, TP2.1; no longer C16.2
- net GND: now also C16.2; no longer C16.1
Other:
- moved on the sheet: C16

Commit message: Cleanup
Connections:
- net GPIO1: no longer JP3.1 (A)
- net GPIO2: no longer U5.3 (SCLK)
- net GPIO23: now also JP3.1 (A)
- net GPIO24: now also R15.2, R16.1, U5.5 (DI)
- net GPIO25: now also JP2.2 (B)
- net GPIO29: now also U5.3 (SCLK)
- net GPIO3: no longer R15.2, R16.1, U5.5 (DI)
- net GPIO4: no longer JP2.2 (B)
Other:
- moved on the sheet: C37, C38, C39, C40, JP1, JP2, JP3, PWR_LED1, R10, R11, R12, R14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
