File: RP2350 Dev Board.kicad_pcb (KiCad board)
At the start: 4 copper layers, 77 x 20.8 mm, 108 parts, among them U2 SM03B-SRSS-TB(LF)(SN)(P), U4 W25Q128

Commit message: Re-did schematic
Parts:
- turned C10 to -90 degrees
- turned C11 to 0 degrees
- turned C12 to -90 degrees
- turned C13 to -90 degrees
- turned C14 to -90 degrees
- turned C36 to 0 degrees
- turned C8 to 0 degrees
- turned C9 to 0 degrees
- turned L2 to 90 degrees
- turned R1 to 180 degrees
- turned R2 to 180 degrees
- turned R28 to 180 degrees
- turned R3 to 180 degrees
- turned R4 to 90 degrees
Connections:
- net QSPI_SCLK renamed Net-(U1-QSPI_SCLK)
- net QSPI_SD0 renamed Net-(U1-QSPI_SD0)
- net QSPI_SD1 renamed Net-(U1-QSPI_SD1)
- net QSPI_SD2 renamed Net-(U1-QSPI_SD2)
- net QSPI_SD3 renamed Net-(U1-QSPI_SD3)
- net QSPI_SS renamed Net-(U1-QSPI_SS)
- net SWCLK renamed Net-(U1-SWCLK)
- net SWD renamed Net-(U1-SWDIO)
- net XIN renamed Net-(U1-XIN)
- C10 pad 1: 1V1 -> GND
- C10 pad 2: GND -> 1V1
- C11 pad 1: Net-(U1-VREG_AVDD) -> GND
- C11 pad 2: GND -> Net-(U1-VREG_AVDD)
- C12 pad 1: 3V3 -> GND
- C12 pad 2: GND -> 3V3
- C13 pad 1: 1V1 -> GND
- C13 pad 2: GND -> 1V1
- C14 pad 1: 3V3 -> GND
- C14 pad 2: GND -> 3V3
- C36 pad 1: 3V3 -> GND
- C36 pad 2: GND -> 3V3
- C8 pad 1: 3V3 -> GND
- C8 pad 2: GND -> 3V3
- C9 pad 1: 3V3 -> GND
- C9 pad 2: GND -> 3V3
- L2 pad 1: /VREG_LX -> 1V1
- L2 pad 2: 1V1 -> /VREG_LX
- R1 pad 1: Net-(USB1-CC1) -> GND
- R1 pad 2: GND -> Net-(USB1-CC1)
- R2 pad 1: USB2_D- -> Net-(U1-USB_DM)
- R2 pad 2: USB_D- -> USB2_D-
- R28 pad 1: XOUT -> Net-(C17-Pad1)
- R28 pad 2: Net-(C17-Pad1) -> Net-(U1-XOUT)
- R3 pad 1: USB2_D+ -> Net-(U1-USB_DP)
- R3 pad 2: USB_D+ -> USB2_D+
- R4 pad 1: Net-(USB1-CC2) -> GND
- R4 pad 2: GND -> Net-(USB1-CC2)
- U1 pad 31: XOUT -> Net-(U1-XOUT)
- U1 pad 66: USB_D- -> Net-(U1-USB_DM)
- U1 pad 67: USB_D+ -> Net-(U1-USB_DP)
Routing:
- net USB_D-: track 8.65 -> 0.00 mm
- net Net-(U1-USB_DM): track 0.00 -> 8.65 mm
- net USB_D+: track 8.18 -> 0.00 mm
- net Net-(U1-USB_DP): track 0.00 -> 8.18 mm
- net XOUT: track 2.50 -> 0.00 mm
- net Net-(U1-XOUT): track 0.00 -> 2.50 mm

Commit message: Updated footprints, more basic parts
Parts:
- removed L2: ~, RP2350 Dev Board:IND-SMD_L2.0-W1.6_AOTA-B201610S3R3-101-T
- added L1: ~, RP2350 Dev Board:IND-SMD_L2.0-W1.6_AOTA-B201610S3R3-101-T, F.Cu at (138.0, 98.5)
- C37, C38, C39, C40: footprint PCM_JLCPCB:R_0402 -> PCM_JLCPCB:C_0603
- PWR_LED1: value ~ -> Red; footprint RP2350 Dev Board:LED0402-RD -> PCM_JLCPCB:D_0603
- R5: footprint PCM_JLCPCB:R_0603 -> PCM_JLCPCB:R_0402
- R7, R8: footprint PCM_JLCPCB:R_0402 -> PCM_JLCPCB:R_0603
- U2: value SM03B-SRSS-TB(LF)(SN)(P) -> HC-1.0-3PWT
- moved PWR_LED1 6.47 mm to (111.8, 107.2)
- moved C19 4.39 mm to (135.2, 95.6)
- moved R7 3.83 mm to (132.9, 95.7), turned to 180 degrees
- moved C39 0.87 mm to (118.1, 102.6), turned to -90 degrees
- moved R11 0.65 mm to (118.8, 104.8)
- moved C37 0.48 mm to (119.3, 102.9), turned to -90 degrees
- moved U3 0.42 mm to (121.7, 103.4)
- moved R4 0.38 mm to (117.0, 103.4)
- moved R5 0.37 mm to (125.4, 95.3)
- moved R8 0.34 mm to (127.6, 95.0)
- moved C40 0.33 mm to (124.2, 102.7), turned to -90 degrees
- moved C14 0.09 mm to (148.3, 94.6)
- moved C38 0.08 mm to (125.5, 102.8), turned to -90 degrees
Connections:
- C37 pad 1: GND -> VSYS
- C37 pad 2: VSYS -> GND
- C38 pad 1: GND -> 3V3
- C38 pad 2: 3V3 -> GND
- C39 pad 1: GND -> VSYS
- C39 pad 2: VSYS -> GND
- C40 pad 1: GND -> 3V3
- C40 pad 2: 3V3 -> GND
Routing:
- net VBUS: track 32.2 -> 25.0 mm
- net Net-(PWR_LED1-Pad1): track 1.74 -> 8.09 mm
- net Net-(U1-ADC_AVDD): track 17.3 -> 12.3 mm
- net ADC_VREF: track 7.54 -> 10.4 mm
- net Net-(Boot1-Pad1): track 8.37 -> 9.23 mm
- net 3V3_EN: track 12.9 -> 13.6 mm
- net 3V3: track 20.9 -> 20.7 mm, vias 11 -> 10
- net VSYS: vias 4 -> 6

Commit message: Added wifi and PSRAM
Parts:
- added H1: PM254V-12-08-H85_C2834799, EasyEDA:HDR-TH_8P-P2.54-V-F-R2-C4-S2.54, F.Cu at (202.7, 100.2)
- added R10: 10kΩ, PCM_JLCPCB:R_0402, F.Cu at (196.8, 107.5)
- added R13: 10kΩ, PCM_JLCPCB:R_0402, F.Cu at (196.8, 109.4)
- added R9: 10kΩ, PCM_JLCPCB:R_0402, F.Cu at (196.8, 105.7)

Commit message: Super version
Parts:
- added C20: 100nF, RP2350 Dev Board:C0402, F.Cu at (215.0, 89.9)
- added R14: 10kΩ, PCM_JLCPCB:R_0402, F.Cu at (218.2, 89.8)
- added U6: ESP-PSRAM32, Package_SO:SOIC-8_3.9x4.9mm_P1.27mm, F.Cu at (121.7, 77.2)
- U4: value W25Q128 -> ESP-PSRAM64H

Commit message: Super version
Parts:
- removed 3V31, 3V3_EN1, ADC_VREF1, GND1, GND2, GND3, GND4 (x2), GND6, GPI10, GPIO0, GPIO1 (x8), GPIO11, GPIO12, GPIO13, GPIO15, GPIO16, GPIO17, GPIO18, GPIO19, GPIO2, GPIO21 (x2), GPIO22, GPIO24, GPIO25, GPIO26, GPIO27, GPIO28, GPIO29, GPIO3, GPIO30, GPIO32, GPIO34, GPIO35, GPIO36, GPIO37, GPIO38, GPIO39, GPIO4, GPIO40, GPIO41, GPIO42, GPIO43, GPIO44, GPIO45, GPIO46, GPIO5, GPIO7, GPIO8, RUN1, VBUS1, VSYS1: Castellated Pad, My Stuff:Castellated Pad
- removed C20: 100nF, RP2350 Dev Board:C0402
- removed H1: PM254V-12-08-H85_C2834799, EasyEDA:HDR-TH_8P-P2.54-V-F-R2-C4-S2.54
- removed R13: 10kΩ, PCM_JLCPCB:R_0402
- removed U2: HC-1.0-3PWT, EasyEDA:CONN-SMD_SM03B-SRSS-TB-LF-SN-P
- added J1: Conn_01x32_MountingPin, Custom:Pads_1x33_P2.54mm_Vertical_2, F.Cu at (110.9, 92.6)
- added J2: Conn_01x03_Pin, Connector_PinHeader_2.54mm:PinHeader_1x03_P2.54mm_Vertical, F.Cu at (174.8, 98.2)
- added J3: Conn_01x32_MountingPin, Custom:Pads_1x33_P2.54mm_Vertical, F.Cu at (110.9, 110.4)
- added JP1: SolderJumper_2_Open, Jumper:SolderJumper-2_P1.3mm_Open_Pad1.0x1.5mm, B.Cu at (111.6, 108.2)
- added JP2: SolderJumper_2_Open, Jumper:SolderJumper-2_P1.3mm_Open_Pad1.0x1.5mm, B.Cu at (124.2, 108.2)
- added JP3: SolderJumper_2_Open, Jumper:SolderJumper-2_P1.3mm_Open_Pad1.0x1.5mm, B.Cu at (115.4, 108.2)
- added R15: 470Ω, PCM_JLCPCB:R_0402, F.Cu at (180.7, 94.5)
- added R16: 10kΩ, PCM_JLCPCB:R_0402, F.Cu at (180.7, 95.8)
- added U5: RPI Radio Module 2, Custom:rpi_rmc20452t, F.Cu at (190.3, 101.5)
- U4: value ESP-PSRAM64H -> Winbond W25Q128JVSIQ
- U6: moved to B.Cu
- moved R14 86.7 mm to (133.2, 107.2)
- moved U6 27.6 mm to (131.1, 103.2), turned to 90 degrees
- moved R9 18.1 mm to (180.2, 98.5), turned to 180 degrees
- moved R10 17.1 mm to (180.2, 103.0), turned to 180 degrees
- moved R8 4.98 mm to (132.6, 95.5), turned to 180 degrees
- moved C19 2.44 mm to (137.6, 96.0)
- moved R7 2.41 mm to (135.3, 95.9)
- moved C7 1.47 mm to (153.8, 97.0)
- moved PWR_LED1 0.64 mm to (112.3, 106.9)
- moved C17 0.28 mm to (158.0, 100.5)
- moved C18 0.28 mm to (158.0, 102.7)
- moved X1 0.28 mm to (160.7, 101.7)
- moved R28 0.25 mm to (155.6, 100.9)
- moved C5 0.15 mm to (155.8, 99.9)
- moved C14 0.15 mm to (148.3, 94.8)
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Connections:
- R10 pad 2: 3V3 -> GND
- R14 pad 1: GPIO47/ADC7 -> Net-(JP1-A)
- R9 pad 1: 3V3 -> Net-(JP2-A)
- R9 pad 2: Net-(H1-CS) -> GND
- U1 pad 33: Net-(U1-SWCLK) -> SWCLK
- U1 pad 34: Net-(U1-SWDIO) -> SWDIO
- U1 pad 70: Net-(U1-QSPI_SD3) -> QSPI_SD3
- U1 pad 71: Net-(U1-QSPI_SCLK) -> QSPI_SCLK
- U1 pad 72: Net-(U1-QSPI_SD0) -> QSPI_SD0
- U1 pad 73: Net-(U1-QSPI_SD2) -> QSPI_SD2
- U1 pad 74: Net-(U1-QSPI_SD1) -> QSPI_SD1
- U4 pad 2: Net-(U1-QSPI_SD1) -> QSPI_SD1
- U4 pad 3: Net-(U1-QSPI_SD2) -> QSPI_SD2
- U4 pad 5: Net-(U1-QSPI_SD0) -> QSPI_SD0
- U4 pad 6: Net-(U1-QSPI_SCLK) -> QSPI_SCLK
- U4 pad 7: Net-(U1-QSPI_SD3) -> QSPI_SD3
- U6 pad 1: GPIO47/ADC7 -> Net-(JP1-A)
Routing:
- net Net-(JP3-B): track 0.00 -> 83.2 mm, vias 0 -> 1
- net GPIO2: track 29.3 -> 112.5 mm, vias 0 -> 1
- net GPIO3: track 26.6 -> 107.4 mm, vias 0 -> 3
- net Net-(JP2-A): track 0.00 -> 66.2 mm, vias 0 -> 1
- net GPIO36: track 11.3 -> 49.8 mm
- net GPIO37: track 9.20 -> 46.1 mm
- net GPIO42/ADC2: track 5.52 -> 37.4 mm
- net GPIO39: track 5.08 -> 36.9 mm
- net GPIO38: track 7.11 -> 38.8 mm
- net GPIO41/ADC1: track 5.03 -> 35.4 mm
- net GPIO40/ADC0: track 4.67 -> 34.8 mm
- net GPIO35: track 13.4 -> 42.9 mm
- net Net-(U1-SWCLK): track 29.6 -> 0.00 mm
- net Net-(U1-SWDIO): track 29.0 -> 0.00 mm
- net QSPI_SD1: track 0.00 -> 28.9 mm, vias 0 -> 1
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Other:
- board size 77 x 20.8 mm -> 84.8 x 23.7 mm
- board text added: "3V3"
- board text added: "3VEN"
- board text added: "40A0"
- board text added: "41A1"
- board text added: "42A2"
- board text added: "43A3"
- board text added: "44A4"
- board text added: "45A5"
- board text added: "46A6"
- board text added: "47A7"
- board text added: "<Pico 1"
- board text added: "GND"
- board text added: "GP0"
- board text added: "GP1"
- board text added: "GP10"
- board text added: "GP11"
- board text added: "GP12"
- board text added: "GP13"
- board text added: "GP14"
- board text added: "GP15"
- board text added: "GP16"
- board text added: "GP17"
- board text added: "GP18"
- board text added: "GP19"
- board text added: "GP2"
- board text added: "GP20"
- board text added: "GP21"
- board text added: "GP22"
- board text added: "GP23"
- board text added: "GP24"
- board text added: "GP25"
- board text added: "GP26"
- board text added: "GP27"
- board text added: "GP28"
- board text added: "GP29"
- board text added: "GP3"
- board text added: "GP30"
- board text added: "GP31"
- board text added: "GP32"
- board text added: "GP33"
- board text added: "GP34"
- board text added: "GP35"
- board text added: "GP36"
- board text added: "GP37"
- board text added: "GP38"
- board text added: "GP39"
- board text added: "GP4"
- board text added: "GP5"
- board text added: "GP6"
- board text added: "GP7"
- board text added: "GP8"
- board text added: "GP9"
- board text added: "JP1 PSRAM JP2/JP3 WIFI"
- board text added: "Pico 2 >"
- board text added: "RUN"
- board text added: "SWCLK"
- board text added: "SWDIO"
- board text added: "VBUS"
- board text added: "VREF"
- board text added: "VSYS"

Commit message: Cleanup
Parts:
- moved R7 0.35 mm to (135.3, 95.5)
Routing:
- net ADC_VREF: track 13.4 -> 12.1 mm
- net GND: vias 58 -> 57
Other:
- board text removed: "<Pico 1"
- board text removed: "Pico 2 >"

Commit message: final cleanup
Parts:
- J1: footprint Custom:Pads_1x33_P2.54mm_Vertical_2 -> Connector_PinHeader_2.54mm:PinHeader_1x32_P2.54mm_Vertical
- J3: footprint Custom:Pads_1x33_P2.54mm_Vertical -> Connector_PinHeader_2.54mm:PinHeader_1x32_P2.54mm_Vertical
