File: pico-stretch.kicad_pcb (KiCad board)
At the start: 4 copper layers, 84.8 x 23.7 mm, 64 parts, among them J1 Conn_01x32_MountingPin, J2 Conn_01x03_Pin, J3 Conn_01x32_MountingPin, U4 Winbond W25Q128JVSIQ, U5 RPI Radio Module 2, U6 ESP-PSRAM32

Commit message: Fixes, 3v3 front pour, change to signal/gnd/gnd/signal stackup
Parts:
- moved R14 19.3 mm to (113.9, 107.2), turned to -90 degrees
- moved R12 1.78 mm to (122.2, 106.6)
Routing:
- net 3V3: track 25.7 -> 15.5 mm, vias 13 -> 2
- net GPIO8: track 12.3 -> 15.3 mm
- net GPIO9: track 10.2 -> 12.6 mm
- net Net-(PWR_LED1-Pad1): track 2.60 -> 1.61 mm
- net GPIO20: track 23.8 -> 24.6 mm
- net RUN: track 47.9 -> 48.5 mm
- net GPIO18: track 25.3 -> 24.8 mm
- net Net-(U1-ADC_AVDD): track 10.3 -> 10.1 mm, vias 0 -> 2
- net GND: vias 57 -> 117
- added copper zone on In2.Cu, net GND
- removed copper zone on In2.Cu, net 3V3

Commit message: Fixes after review
Parts:
- added C21: 100nF, PCM_JLCPCB:C_0402, F.Cu at (192.2, 110.5)
- added C22: 100nF, PCM_JLCPCB:C_0402, F.Cu at (133.5, 98.0)
- added C23: 100nF, PCM_JLCPCB:C_0402, F.Cu at (180.9, 107.6)
- added C24: 4.7nF, PCM_JLCPCB:C_0603, F.Cu at (180.5, 105.3)
- moved D2 0.67 mm to (134.6, 97.5), turned to -90 degrees
- moved C16 0.06 mm to (136.9, 101.7)
Routing:
- net GND: track 2.80 -> 10.5 mm, vias 117 -> 136
- net 3V3: track 15.5 -> 21.0 mm, vias 2 -> 3
- net GPIO24: track 60.9 -> 61.9 mm
- net Net-(JP2-A): track 27.4 -> 28.3 mm
- net GPIO37: track 46.1 -> 46.6 mm
